Commit message: Finished Example

File: urdf/robot_on_rail.xacro (robot description, xacro)
@@ -2,9 +2,12 @@
 <robot name="robot_on_rail" xmlns:xacro="http://ros.org/wiki/xacro">
   <!-- Get the macros we will need -->
-  <xacro:include filename="$(find abb_irb4400)/urdf/irb4400l_30_243_macro.xacro"/>
+  <xacro:include filename="$(find abb_irb4400_support)/urdf/irb4400l_30_243_macro.xacro"/>
   <xacro:include filename="$(find timing_example)/urdf/robot_transport_unit_macro.xacro"/>
+  <xacro:include filename="$(find timing_example)/urdf/lathe_macro.xacro"/>
   <!-- Import instances of the macros -->
   <xacro:abb_irb4400l_30_243 prefix="robot_"/>
   <xacro:robot_transport_unit prefix="rail_"/>
+  <xacro:lathe prefix="lathe1_"/>
+  <xacro:lathe prefix="lathe2_"/>
   <!-- Extra links -->
   <link name="world"/>
@@ -16,7 +19,17 @@
   </joint>
   <joint name="robot_to_rail" type="fixed">
-    <origin xyz="0 -0 -0.390" rpy="0 0 0"/>
+    <origin xyz="0 -0 -0.390" rpy="0 0 3.14"/>
     <parent link="rail_tool0"/>
     <child link="robot_base_link"/>
   </joint>
+  <joint name="world_to_lathe1" type="fixed">
+    <origin xyz="2.5 0 0" rpy="0 0 0"/>
+    <parent link="world"/>
+    <child link="lathe1_base_link"/>
+  </joint>
+  <joint name="world_to_lathe2" type="fixed">
+    <origin xyz="-2.5 0 0" rpy="0 0 0"/>
+    <parent link="world"/>
+    <child link="lathe2_base_link"/>
+  </joint>
 </robot>

File: urdf/robot_transport_unit_macro.xacro (robot description, xacro)
@@ -7,9 +7,9 @@
   <xacro:macro name="robot_transport_unit" params="prefix">
     <!-- Top-level links -->
-    <link name="${prefix}base_link"/>
-    <link name="${prefix}carriage">
+    <link name="${prefix}base_link">
       <visual>
+        <origin xyz="2.5 0.0 0.125" rpy="0.0 0.0 0.0"/>
         <geometry>
-          <mesh filename="package://timing_example/meshes/visual/carriage.stl"/>
+          <box size="6.0 1.0 0.25"/>
         </geometry>
         <material name="${prefix}carriage_visual_material">
@@ -19,7 +19,27 @@
       <!--These collision tags were generated automatically-->
       <collision>
-        <origin xyz="1.67045 0.1215 2.14435" rpy="0  0  ${radians(180)}"/>
+        <origin xyz="2.5 0.0 0.125" rpy="0.0 0.0 0.0"/>
         <geometry>
-          <mesh filename="package://timing_example/meshes/collision/carriage.stl"/>
+          <box size="6.0 1.0 0.25"/>
+        </geometry>
+        <material name="world_collision_material">
+          <color rgba="0.6 0.6 0.6 1"/>
+        </material>
+      </collision>
+    </link>
+    <link name="${prefix}carriage">
+      <visual>
+        <origin xyz="0 0 0.25" rpy="0 0 0"/>
+        <geometry>
+          <box size="0.75 1.25 0.25"/>
+        </geometry>
+        <material name="${prefix}carriage_visual_material">
+          <color rgba="0.75 0.2 0.2 1"/>
+        </material>
+      </visual>
+      <collision>
+        <origin xyz="0 0 0.25" rpy="0 0 0"/>
+        <geometry>
+          <box size="0.75 1.25 0.25"/>
         </geometry>
         <material name="world_collision_material">
@@ -40,5 +60,5 @@
       <parent link="${prefix}carriage"/>
       <child link="${prefix}tool0"/>
-      <origin xyz="01.26735 00.28829 02.13236" rpy="0 0 0"/>
+      <origin xyz="0.0 0.0 0.75" rpy="0 0 0"/>
     </joint>
   </xacro:macro>

File: urdf/two_robots.xacro (robot description, xacro)
@@ -6,6 +6,9 @@
   <xacro:abb_irb4400l_30_243 prefix="robot0_"/>
   <xacro:abb_irb4400l_30_243 prefix="robot1_"/>
+  <xacro:lathe prefix="lathe1_"/>
+  <xacro:lathe prefix="lathe2_"/>
   <!-- Extra links -->
   <link name="world"/>
+  <!-- Connect the imported macro instances -->
   <joint name="robot1_to_world" type="fixed">
     <origin xyz="0 -2.000 0" rpy="0 0 0"/>
@@ -18,3 +21,13 @@
     <child link="robot2_base_link"/>
   </joint>
+  <joint name="world_to_lathe1" type="fixed">
+    <origin xyz="2.5 0 0" rpy="0.0.0"/>
+    <parent link="world"/>
+    <child link="lathe1_base_link"/>
+  </joint>
+  <joint name="world_to_lathe2" type="fixed">
+    <origin xyz="-2.5 0 0" rpy="0.0.0"/>
+    <parent link="world"/>
+    <child link="lathe2_base_link"/>
+  </joint>
 </robot>
